Commit message: zed-wrapper updated

File: zed-ros-wrapper/zed_wrapper/urdf/zed.urdf (robot description, URDF)
Before this commit: robot zed_camera, 5 links, 4 joints
Links:
- added link base_link
- link zed_camera_center: geometry visual mesh filename=package://zed_wrapper/urdf/models/ZED.stl
Joints:
- added joint zed_camera_center_joint: type fixed, parent base_link, child zed_camera_center, origin xyz=0 0 0 rpy=0 0 0

File: zed-ros-wrapper/zed_wrapper/urdf/zedm.urdf (robot description, URDF)
Before this commit: robot zedm_camera, 6 links, 5 joints
Links:
- removed link imu_link
- added link base_link
- added link zed_imu_link
- link zed_camera_center: geometry visual mesh filename=package://zed_wrapper/urdf/models/ZEDM.stl
Joints:
- added joint zed_camera_center_joint: type fixed, parent base_link, child zed_camera_center, origin xyz=0 0 0 rpy=0 0 0
- joint imu_link_joint: child imu_link -> zed_imu_link
